File: Hardware/Basic/Bottom/Fyre-BASIC-BOTtom.brd (EAGLE design)
At the start: 33 x 33 mm, 38 parts, among them U3 PCF8523, Y2 32.7680kHz

Commit message: Completed the top board
Changed lines of the file:
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@@
 <drawing>
 <settings>
-<setting alwaysvectorfont="no"/>
+<setting alwaysvectorfont="yes"/>
 <setting verticaltext="up"/>
 </settings>
-<grid distance="0.1" unitdist="mil" unit="mil" style="lines" multiple="1" display="yes" altdistance="5" altunitdist="mil" altunit="mil"/>
+<grid distance="0.1" unitdist="mil" unit="mm" style="lines" multiple="1" display="yes" altdistance="5" altunitdist="mil" altunit="mil"/>
 <layers>
 <layer number="1" name="Top" color="4" fill="1" visible="yes" active="yes"/>
@@
 </element>
 <element name="R16" library="LinnesLab-Passives" package="R0603" package3d_urn="urn:adsk.eagle:package:15661944/2" value="" x="19.1262" y="29.850075" smashed="yes">
-<attribute name="NAME" x="18.4912" y="30.485075" size="0.7112" layer="25"/>
+<attribute name="NAME" x="18.21941875" y="30.75685625" size="0.7112" layer="25"/>
 <attribute name="VALUE" x="18.4912" y="27.945075" size="1.27" layer="27"/>
 </element>
@@
 <wire x1="22.63394375" y1="19.17519375" x2="22.1236625" y2="19.685475" width="0.1524" layer="1"/>
 <wire x1="22.1236625" y1="20.208503125" x2="22.1236625" y2="19.685475" width="0.1524" layer="1"/>
-<wire x1="30.54858125" y1="22.54593125" x2="30.484184375" y2="22.481534375" width="0.1524" layer="1"/>
 <wire x1="30.834709375" y1="5.687059375" x2="31.866840625" y2="5.687059375" width="0.1524" layer="1"/>
 <wire x1="31.866840625" y1="5.687059375" x2="31.993840625" y2="5.814059375" width="0.1524" layer="1"/>
@@
 <wire x1="25.168859375" y1="13.921740625" x2="25.168859375" y2="13.26641875" width="0.1524" layer="16"/>
 <contactref element="C1" pad="1"/>
-<wire x1="22.63394375" y1="16.5979375" x2="22.44785" y2="16.41184375" width="0.1524" layer="1"/>
-<wire x1="30.559640625" y1="24.003" x2="30.559640625" y2="22.556990625" width="0.1524" layer="1"/>
-<wire x1="30.559640625" y1="22.556990625" x2="30.484184375" y2="22.481534375" width="0.1524" layer="1"/>
+<wire x1="30.559640625" y1="24.003" x2="30.5545625" y2="23.997921875" width="0.1524" layer="1"/>
+<wire x1="30.5545625" y1="23.997921875" x2="30.5545625" y2="22.5519125" width="0.1524" layer="1"/>
+<wire x1="30.484184375" y1="22.481534375" x2="30.5545625" y2="22.5519125" width="0.1524" layer="1"/>
 <wire x1="30.559640625" y1="24.003" x2="30.55845" y2="24.001809375" width="0.1524" layer="1"/>
 <wire x1="30.55845" y1="24.001809375" x2="25.91696875" y2="24.001809375" width="0.1524" layer="1"/>
