File: Hardware/Basic/Top/Fyre-BASIC-TOP.brd (EAGLE design)
At the start: 38 x 38 mm, 66 parts, among them SW1 SWITCH.MOM, SW2 SWITCH.MOM, SW5 SWITCH.MOM, U2 NRF52832_MODULE_MDBT42, U4 PCF8523, U5 FT231XS

Commit message: Completed the top board
Parts:
- removed C19: 2.2uF, LinnesLab-Passives:C0402
- removed C20, C21: 4.7u, LinnesLab-Passives:C0603
- removed C22: 100n, LinnesLab-Passives:C0603
- removed C23, C24: 47p, LinnesLab-Passives:C0603
- removed CHRG2: MCP73831, LinnesLab-Power:SOT23-5
- removed CORTEX1: CORTEX_DEBUG_PTH, LinnesLab-Connectors:2X5-PTH-1.27MM
- removed D4, D5: (no value), LinnesLab-DiscreteSemi:USC
- removed JP2: (no value), LinnesLab-Switches:SMT-JUMPER_2_NO_SILK
- removed L2: 10u, LinnesLab-Passives:L0603
- removed LDO2: MIC5504, LinnesLab-Power:SOT23-5
- removed LED5: RED, LinnesLab-LED:LED-0603
- removed LED6: YELLOW, LinnesLab-LED:LED-0603
- removed R18: 27, LinnesLab-Passives:R0603
- removed R19, R20: 1k, LinnesLab-Passives:R0603
- removed SD2: (no value), LinnesLab-Connectors:MICROSD
- removed SW5: SWITCH.MOM, LinnesLab-Switches:TACTILE_SWITCH_SMD_6.2MM_TALL
- removed U4: PCF8523, LinnesLab-Clocks:SO8
- removed U5: FT231XS, LinnesLab-DigitalIC:SSOP20_L
- removed USB2: USB.MICRO-BIGGERPADS, LinnesLab-Connectors:USB-MICRO-01.BIGGERPADS
- removed XTAL2: 32.768kHz, LinnesLab-Clocks:2-SMD.NOLEAD.2.0MMTO1.2MM
- removed XTAL3: 32.7680kHz, LinnesLab-Clocks:2-SMD.NOLEAD.2.0MMTO1.2MM
- added C1: 1u, LinnesLab-Passives:C0603
- added C3, C4: (no value), LinnesLab-Passives:C0603
- added CHRG1: MCP73831, LinnesLab-Power:SOT23-5
- added D2, D3: (no value), LinnesLab-DiscreteSemi:USC
- added DEBUG1: CORTEX_DEBUG_PTH, LinnesLab-Connectors:2X5-PTH-1.27MM
- added JP1: (no value), LinnesLab-Switches:SMT-JUMPER_2_NO_SILK
- added L1: 10u, LinnesLab-Passives:L0603
- added LDO1: MIC5504, LinnesLab-Power:SOT23-5
- added LED1: RED, LinnesLab-LED:LED-0603
- added LED2: BLUE, LinnesLab-LED:LED-0603
- added R10: 27, LinnesLab-Passives:R0603
- added R16: 0, LinnesLab-Passives:R0603
- added SD1: (no value), LinnesLab-Connectors:MICROSD
- added U1: NRF52832_MODULE_MDBT42, LinnesLab-Microcontrollers:BLE_MODULE_RAYTAC_MDBT42
- added USB1: USB.MICRO-BIGGERPADS, LinnesLab-Connectors:USB-MICRO-01.BIGGERPADS
- added XTAL1: 32.768kHz, LinnesLab-Clocks:2-SMD.NOLEAD.2.0MMTO1.2MM
- C10, C11: value 300p -> 47p
- C12: value 10u -> 100n; device LinnesLab-Passives:C0805 -> LinnesLab-Passives:C0603
- C13: value 2.2uF -> 10uF; device LinnesLab-Passives:C0402 -> LinnesLab-Passives:C0603
- C14: value 100n -> 2.2uF; device LinnesLab-Passives:C0603 -> LinnesLab-Passives:C0402
- C16: value 10uF -> 2.2uF; device LinnesLab-Passives:C0603 -> LinnesLab-Passives:C0402
- C2: value 1u -> 10u; device LinnesLab-Passives:C0603 -> LinnesLab-Passives:C0805
- C5: value 1u -> 4.7u
- C8: value (none) -> 4.7u
- C9: value (none) -> 100n
- J1: device LinnesLab-Connectors:1X06_1.27MM -> LinnesLab-Connectors:1X02
- J2: device LinnesLab-Connectors:1X02 -> LinnesLab-Connectors:1X07_1.27MM
- LED4: value BLUE -> YELLOW
- R1, R2: value 0 -> 10k
- R11: value (none) -> 27
- R12: value 100k -> 10k
- R13, R15: value 100k -> 1k
- R14: value 100k -> 390k
- R17: value 27 -> 0
- R3: value 1k -> 100k
- R5: value 10k -> (none)
- R6: value 10k -> 1k
- R7: value 390k -> 100k
- R8: value 10k -> 100k
- SW2: value SWITCH.MOM -> (none); device LinnesLab-Switches:TACTILE_SWITCH_SMD_6.2MM_TALL -> LinnesLab-Switches:BUTTON-GULLWING
- SW3: value (none) -> SWITCH.MOM; device LinnesLab-Switches:BUTTON-GULLWING -> LinnesLab-Switches:TACTILE_SWITCH_SMD_6.2MM_TALL
- U2: value NRF52832_MODULE_MDBT42 -> FT231XS; device LinnesLab-Microcontrollers:BLE_MODULE_RAYTAC_MDBT42 -> LinnesLab-DigitalIC:SSOP20_L
- moved R9 73.2 mm to (34.6, 11.4), turned to 180 degrees
- moved R2 67.7 mm to (3.76, 28.8), turned to 270 degrees
- moved R1 64.6 mm to (1.75, 28.8), turned to 270 degrees
- moved R8 64.0 mm to (2.01, 21.3), turned to 90 degrees
- moved R5 43.3 mm to (2.46, 12.3), flipped to the bottom, turned to 180 degrees
- moved D1 42.2 mm to (8.28, 3.56), flipped to the bottom, turned to 270 degrees
- moved C14 40.7 mm to (9.58, 21.9), turned to 180 degrees
- moved U2 33.9 mm to (7.18, 6.01), turned to 270 degrees
- moved SW2 33.6 mm to (35.0, 35.2)
- moved LED4 31.9 mm to (16.4, 10.3), turned to 180 degrees
- moved LED3 31.6 mm to (16.4, 8.09), turned to 180 degrees
- moved SW3 31.1 mm to (32.2, 4.08), turned to 180 degrees
- moved R3 30.8 mm to (13.1, 9.03), flipped to the bottom, turned to 270 degrees
- moved R6 30.3 mm to (35.3, 23.1), turned to 90 degrees
- moved R12 28.8 mm to (14.5, 21.7), turned to 270 degrees
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Connections:
- removed net A4/BATT: R13.1, R14.2, U2.5
- removed net A6/TIA: U2.7
- removed net A7/PPG: U2.8
- removed net D29/LED.CTRL: U2.6
- removed net N$18: J1.5
- removed net N$19: U4.2, XTAL3.P$1
- removed net N$20: U4.1, XTAL3.P$2
- removed net N$21: J1.4
- removed net N$6: J1.6
- removed net SW1: SW5.A1
- removed net TDX.FT: R1.1
- removed net VBAT: U4.3
- new net A4/PPG: J2.7, U1.5
- new net A5/TIA: J2.6, U1.6
- new net A7/BATT: R7.1, R8.2, U1.8
- new net D30/LED.CTRL: J2.5, U1.7
- net !CTS: now also JP1.2, U2.9; no longer JP2.2, U5.9
- net 3.3V: now also C18.2, C2.2, C7.1, D3.-, DEBUG1.1, J2.4, LDO1.5, LED3.A, LED4.A, R1.2, R2.2, SD1.4, U1.11, U2.14, U2.3; no longer C19.2, C2.1, C22.2, C6.1, CORTEX1.1, D1.-, LDO2.5, LED5.A, LED6.A, R15.2, R5.2, R8.2, SD2.4, U2.11, U4.8, U5.14, U5.3
- net CD2: now also SD1.CD2; no longer SD2.CD2
- net D11/SW1: now also U1.25; no longer U2.25
- net D15/SW2: now also SW3.A1, U1.29; no longer SW2.A1, U2.29
- net D16/CS.OLED: now also U1.30; no longer U2.30
- net D27/CHRG.STATUS: now also CHRG1.1, R3.1, U1.4; no longer CHRG2.1, R12.1, U2.4
- net D3/RESET.OLED: now also U1.16; no longer U2.16
- net D4/DC.OLED: now also U1.17; no longer U2.17
- net D5/CD1: now also SD1.CD1, U1.18; no longer SD2.CD1, U2.18
- net D7/SD.SC: now also SD1.2, U1.20; no longer SD2.2, U2.20
- net DFU: now also SW2.3, U1.34; no longer SW3.3, U2.34
- net DTR: now also C9.1, U2.1; no longer C14.1, U5.1
- net FRST: now also U1.38; no longer U2.38
- net FT3V3: now also U2.13; no longer U5.13
- net GND: now also C1.2, C10.1, C13.1, C15.1, C2.1, C3.1, C4.2, C6.1, C8.2, CHRG1.2, DEBUG1.3, DEBUG1.5, DEBUG1.7, DEBUG1.9, J1.1, J2.3, JP1.1, LDO1.2, LED1.C, LED2.C, R12.1, R14.2, R5.1, R8.1, SD1.6, SD1.MT1, SD1.MT2, SW2.1, SW3.B1, SW3.B2, U1.1, U1.12, U1.24, U1.39, U2.16, U2.6, USB1.5; no longer C10.2, C16.1, C19.1, C2.2, C20.2, C21.1, C22.1, C23.2, C24.1, C6.2, C8.1, C9.2, CHRG2.2, CORTEX1.3, CORTEX1.5, CORTEX1.7, CORTEX1.9, J2.1, JP2.1, LDO2.2, LED3.C, LED4.C, R11.1, R14.1, R15.1, R6.1, R7.2, SD2.6, SD2.MT1, SD2.MT2, SW2.B1, SW2.B2, SW3.1, SW5.B1, SW5.B2, U2.1, U2.12, U2.24, U2.39, U4.4, U5.16, U5.6, USB2.5
- net LED1: now also R4.2, U1.31; no longer R3.2, U2.31
- net LED2: now also R6.2, U1.33; no longer R4.2, U2.33
- net MISO: now also SD1.7, U1.28; no longer SD2.7, U2.28
- net MOSI: now also SD1.3, U1.27; no longer SD2.3, U2.27
- net N$1: now also R12.2; no longer R6.2
- net N$10: now also LED2.A, R6.1; no longer LED4.A, R4.1
- net N$11: now also L1.1, U1.10; no longer L2.1, U2.10
- net N$12: now also C1.1, L1.2, U1.9; no longer C7.1, L2.2, U2.9
- net N$13: now also C13.2; no longer C16.2
- net N$14: now also DEBUG1.8; no longer CORTEX1.8
- net N$15: now also C15.2; no longer C18.2
- net N$16: now also C4.1, U1.14, XTAL1.P$2; no longer C9.1, U2.14, XTAL2.P$2
- net N$17: now also CHRG1.5, R5.2; no longer CHRG2.5, R11.2
- net N$2: now also R14.1; no longer R7.1
- net N$23: now also R10.2, U2.12; no longer R17.2, U5.12
- net N$24: now also R11.2, U2.11; no longer R18.2, U5.11
- net N$25: now also LED3.C, R13.2; no longer LED5.C, R19.2
- net N$26: now also LED4.C, R15.2; no longer LED6.C, R20.2
- net N$3: now also C16.2; no longer C13.2
- net N$4: now also C3.2, U1.13, XTAL1.P$1; no longer C8.2, U2.13, XTAL2.P$1
- net N$5: now also C16.1; no longer C13.1
- net N$7: now also C14.2; no longer C15.2
- net N$8: now also C14.1; no longer C15.1
- net N$9: now also LED1.A, R4.1; no longer LED3.A, R3.1
- net P0.09/NFC1: now also U1.22; no longer C11.1, U2.22
- net P0.10/NFC2: now also U1.23; no longer C10.1, U2.23
- net RESET: now also C9.2, D3.+, DEBUG1.10, R9.1, U1.35; no longer C14.2, CORTEX1.10, D1.+, R5.1, U2.35
- net RXD.FT: now also R17.1, U2.4; no longer R2.1, U5.4
- net RXD.NRF: now also R16.2, U1.21; no longer R1.2, U2.21
- net RXLED: now also R13.1, U2.17; no longer R19.1, U5.17
- net SCK: now also SD1.5, U1.26; no longer SD2.5, U2.26
- net SCL: now also J2.2, R2.1, U1.3; no longer R9.1, U2.3, U4.6
- net SDA: now also J2.1, R1.1, U1.2; no longer R8.1, U2.2, U4.5
- net SWCLK: now also DEBUG1.4, U1.36; no longer CORTEX1.4, U2.36
- net SWDIO: now also DEBUG1.2, U1.37; no longer CORTEX1.2, U2.37
- net SWO: now also DEBUG1.6, U1.32; no longer CORTEX1.6, U2.32
- net TXD.FT: now also R16.1, U2.20; no longer U5.20
- net TXD.NRF: now also R17.2, U1.19; no longer R2.2, U2.19
- net TXLED: now also R15.1, U2.10; no longer R20.1, U5.10
- net USB+: now also C11.1, R11.1, USB1.3; no longer C23.1, R18.1, USB2.3
- net USB-: now also C10.2, R10.1, USB1.2; no longer C24.2, R17.1, USB2.2
- net VIN: now also C6.2, CHRG1.4, D1.-, D2.-, LDO1.1, LDO1.3, R3.2; no longer C21.2, CHRG2.4, D4.-, D5.-, LDO2.1, LDO2.3, R12.2
- net VLIPO: now also C8.1, CHRG1.3, D1.+, J1.2, R7.2; no longer C20.1, CHRG2.3, D4.+, J2.2, R13.2
- net V_USB: now also D2.+, U2.15, USB1.1; no longer D5.+, U5.15, USB2.1
Routing:
- net GND: track 0.00 -> 69.1 mm, vias 0 -> 26
- net D27/CHRG.STATUS: track 0.00 -> 37.1 mm, vias 0 -> 3
- net D7/SD.SC: track 0.00 -> 34.9 mm, vias 0 -> 1
- net DTR: track 0.00 -> 34.8 mm, vias 0 -> 2
- net MOSI: track 0.00 -> 33.2 mm, vias 0 -> 2
- net RESET: track 0.00 -> 32.3 mm, vias 0 -> 3
- net SCK: track 0.00 -> 29.4 mm, vias 0 -> 2
- net TXD.NRF: track 0.00 -> 28.5 mm, vias 0 -> 2
- net D15/SW2: track 0.00 -> 24.5 mm, vias 0 -> 2
- net USB-: track 0.00 -> 23.9 mm, vias 0 -> 1
- net VLIPO: track 0.00 -> 23.6 mm
- net RXD.NRF: track 0.00 -> 22.8 mm, vias 0 -> 4
- net SDA: track 0.00 -> 22.7 mm, vias 0 -> 1
- net SCL: track 0.00 -> 21.0 mm, vias 0 -> 1
- net D11/SW1: track 0.00 -> 20.9 mm
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- added copper zone on layer 1, net 3.3V
- added copper zone on layer 16, net GND

Commit message: Small changes
Parts:
- renumbered SW4 to RESET
Other:
- board text added: "+"
Changed lines of the file:
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@@
 <drawing>
 <settings>
-<setting alwaysvectorfont="yes"/>
+<setting alwaysvectorfont="no"/>
 <setting verticaltext="up"/>
 </settings>
@@
 <layer number="25" name="tNames" color="7" fill="1" visible="yes" active="yes"/>
 <layer number="26" name="bNames" color="7" fill="1" visible="yes" active="yes"/>
-<layer number="27" name="tValues" color="7" fill="1" visible="no" active="yes"/>
-<layer number="28" name="bValues" color="7" fill="1" visible="no" active="yes"/>
+<layer number="27" name="tValues" color="7" fill="1" visible="yes" active="yes"/>
+<layer number="28" name="bValues" color="7" fill="1" visible="yes" active="yes"/>
 <layer number="29" name="tStop" color="7" fill="3" visible="no" active="yes"/>
 <layer number="30" name="bStop" color="7" fill="6" visible="no" active="yes"/>
@@
 <dimension x1="0" y1="38" x2="0" y2="0" x3="-5.08" y3="19" textsize="1.778" layer="51" dtype="vertical" visible="yes"/>
 <dimension x1="38" y1="38" x2="0" y2="38" x3="19" y3="43.18" textsize="1.778" layer="51" dtype="horizontal" visible="yes"/>
+<text x="4.003040625" y="13.99031875" size="1.778" layer="25">+</text>
+<text x="5.242559375" y="13.9954" size="1.778" layer="26" rot="MR0">+</text>
 </plain>
 <attributes>
@@
 <attribute name="VALUE" x="33.080959375" y="32.9438" size="0.7112" layer="27"/>
 </element>
-<element name="SW4" library="LinnesLab-Switches" package="BUTTON-GULLWING" package3d_urn="urn:adsk.eagle:package:18580190/2" value="" x="34.54654375" y="14.315440625" smashed="yes" rot="R270">
-<attribute name="NAME" x="36.075625" y="15.02918125" size="0.7112" layer="25" rot="R270"/>
+<element name="RESET" library="LinnesLab-Switches" package="BUTTON-GULLWING" package3d_urn="urn:adsk.eagle:package:18580190/2" value="" x="34.54654375" y="14.315440625" smashed="yes" rot="R270">
+<attribute name="NAME" x="36.459165625" y="15.2273" size="0.7112" layer="25" rot="R270"/>
 <attribute name="VALUE" x="32.26054375" y="16.245840625" size="0.7112" layer="27" rot="R270"/>
 </element>
@@
 <contactref element="DEBUG1" pad="9"/>
 <contactref element="SW2" pad="1"/>
-<contactref element="SW4" pad="3"/>
+<contactref element="RESET" pad="3"/>
 <contactref element="U1" pad="24"/>
 <contactref element="U1" pad="1"/>
@@
 <contactref element="C9" pad="2"/>
 <contactref element="DEBUG1" pad="10"/>
-<contactref element="SW4" pad="1"/>
+<contactref element="RESET" pad="1"/>
 <contactref element="U1" pad="35"/>
 <wire x1="35.79875625" y1="26.560771875" x2="36.821440625" y2="25.5380875" width="0.1524" layer="1"/>
