File: Hardware/Basic/Top/Fyre-BASIC-TOP.sch (EAGLE design)
At the start: 66 parts, among them SW1 SWITCH.MOM, SW2 SWITCH.MOM, SW5 SWITCH.MOM, U2 NRF52832_MODULE_MDBT42, U4 PCF8523, U5 FT231XS

Commit message: Completed the top board
Parts:
- removed C19: 2.2uF, LinnesLab-Passives:CAPACITOR0402
- removed C20, C21: 4.7u, LinnesLab-Passives:CAPACITOR0603
- removed C22: 100n, LinnesLab-Passives:CAPACITOR0603
- removed C23, C24: 47p, LinnesLab-Passives:CAPACITOR0603
- removed CHRG2: MCP73831, LinnesLab-Power:MCP73831
- removed CORTEX1: CORTEX_DEBUG_PTH, LinnesLab-Connectors:CORTEX_DEBUG_PTH
- removed D4, D5: (no value), LinnesLab-DiscreteSemi:SCHOTTKY-USC
- removed LDO2: MIC5504, LinnesLab-Power:MIC5504
- removed LED5: RED, LinnesLab-LED:LED0603
- removed LED6: YELLOW, LinnesLab-LED:LED0603
- removed R18: 27, LinnesLab-Passives:RESISTOR0603
- removed R19, R20: 1k, LinnesLab-Passives:RESISTOR0603
- removed SD2: (no value), LinnesLab-Connectors:MICROSD
- removed SW5: SWITCH.MOM, LinnesLab-Switches:SWITCH.MOM
- removed U4: PCF8523, LinnesLab-Clocks:PCF8523
- removed U5: FT231XS, LinnesLab-DigitalIC:FT231XS
- removed USB2: USB.MICRO-BIGGERPADS, LinnesLab-Connectors:USB.MICRO-BIGGERPADS
- removed XTAL3: 32.7680kHz, LinnesLab-Clocks:CRYSTALECS-.327-12.5-12-C-TR
- added C1: 1u, LinnesLab-Passives:CAPACITOR0603
- added C3, C4: (no value), LinnesLab-Passives:CAPACITOR0603
- added CHRG1: MCP73831, LinnesLab-Power:MCP73831
- added D2, D3: (no value), LinnesLab-DiscreteSemi:SCHOTTKY-USC
- added DEBUG1: CORTEX_DEBUG_PTH, LinnesLab-Connectors:CORTEX_DEBUG_PTH
- added LDO1: MIC5504, LinnesLab-Power:MIC5504
- added LED1: RED, LinnesLab-LED:LED0603
- added LED2: BLUE, LinnesLab-LED:LED0603
- added R10: 27, LinnesLab-Passives:RESISTOR0603
- added R16: 0, LinnesLab-Passives:RESISTOR0603
- added SD1: (no value), LinnesLab-Connectors:MICROSD
- added U1: NRF52832_MODULE_MDBT42, LinnesLab-Microcontrollers:NRF52832_MODULE_MDBT42
- added USB1: USB.MICRO-BIGGERPADS, LinnesLab-Connectors:USB.MICRO-BIGGERPADS
- C10, C11: value 300p -> 47p
- C12: value 10u -> 100n; device LinnesLab-Passives:CAPACITOR0805 -> LinnesLab-Passives:CAPACITOR0603
- C13: value 2.2uF -> 10uF; device LinnesLab-Passives:CAPACITOR0402 -> LinnesLab-Passives:CAPACITOR0603
- C14: value 100n -> 2.2uF; device LinnesLab-Passives:CAPACITOR0603 -> LinnesLab-Passives:CAPACITOR0402
- C16: value 10uF -> 2.2uF; device LinnesLab-Passives:CAPACITOR0603 -> LinnesLab-Passives:CAPACITOR0402
- C2: value 1u -> 10u; device LinnesLab-Passives:CAPACITOR0603 -> LinnesLab-Passives:CAPACITOR0805
- C5: value 1u -> 4.7u
- C8: value (none) -> 4.7u
- C9: value (none) -> 100n
- J1: device LinnesLab-Connectors:CONN_061.27MM -> LinnesLab-Connectors:CONN_02
- J2: device LinnesLab-Connectors:CONN_02 -> LinnesLab-Connectors:CONN_07-1.27MM
- LED4: value BLUE -> YELLOW
- R1, R2: value 0 -> 10k
- R11: value (none) -> 27
- R12: value 100k -> 10k
- R13, R15: value 100k -> 1k
- R14: value 100k -> 390k
- R17: value 27 -> 0
- R3: value 1k -> 100k
- R5: value 10k -> (none)
- R6: value 10k -> 1k
- R7: value 390k -> 100k
- R8: value 10k -> 100k
- SW2: value SWITCH.MOM -> (none); device LinnesLab-Switches:SWITCH.MOM -> LinnesLab-Switches:SPST-PTS830GG140-COPY.1-3
- SW3: value (none) -> SWITCH.MOM; device LinnesLab-Switches:SPST-PTS830GG140-COPY.1-3 -> LinnesLab-Switches:SWITCH.MOM
- U2: value NRF52832_MODULE_MDBT42 -> FT231XS; device LinnesLab-Microcontrollers:NRF52832_MODULE_MDBT42 -> LinnesLab-DigitalIC:FT231XS
- renumbered JP2 to JP1, L2 to L1, XTAL2 to XTAL1
Connections:
- removed net A4/BATT: R13.1, R14.2, U2.P0.28/AIN4
- removed net A6/TIA: U2.P0.30/AIN6
- removed net A7/PPG: U2.P0.31/AIN7
- removed net D29/LED.CTRL: U2.P0.29/AIN5
- removed net N$18: J1.5
- removed net N$19: U4.OSCO, XTAL3.1
- removed net N$20: U4.OSCI, XTAL3.2
- removed net N$21: J1.4
- removed net N$6: J1.6
- removed net SW1: SW5.1
- removed net TDX.FT: R1.1
- new net A4/PPG: J2.7, U1.P0.28/AIN4
- new net A5/TIA: J2.6, U1.P0.29/AIN5
- new net A7/BATT: R7.1, R8.2, U1.P0.31/AIN7
- new net D30/LED.CTRL: J2.5, U1.P0.30/AIN6
- net !CTS: now also U2.!CTS; no longer U5.!CTS
- net 3.3V: now also C18.2, C2.2, C7.1, D3.C, DEBUG1.VCC, J2.4, LDO1.OUT, LED3.A, LED4.A, R1.2, R2.2, SD1.VDD, U1.VDD, U2.!RESET, U2.VCCIO; no longer C19.2, C2.1, C22.2, C6.1, CORTEX1.VCC, D1.C, LDO2.OUT, LED5.A, LED6.A, R15.2, R5.2, R8.2, SD2.VDD, U2.VDD, U4.VDD, U5.!RESET, U5.VCCIO
- net CD2: now also SD1.CARD_DETECT1; no longer SD2.CARD_DETECT1
- net D11/SW1: now also U1.P0.11; no longer U2.P0.11
- net D15/SW2: now also SW3.1, U1.P0.15; no longer SW2.1, U2.P0.15
- net D16/CS.OLED: now also U1.P0.16; no longer U2.P0.16
- net D27/CHRG.STATUS: now also CHRG1.STAT, R3.1, U1.P0.27; no longer CHRG2.STAT, R12.1, U2.P0.27
- net D3/RESET.OLED: now also U1.P0.03/AIN1; no longer U2.P0.03/AIN1
- net D4/DC.OLED: now also U1.P0.04/AIN2; no longer U2.P0.04/AIN2
- net D5/CD1: now also SD1.CARD_DETECT, U1.P0.05/AIN3; no longer SD2.CARD_DETECT, U2.P0.05/AIN3
- net D7/SD.SC: now also SD1.CS, U1.P0.07; no longer SD2.CS, U2.P0.07
- net DFU: now also SW2.B, U1.P0.20; no longer SW3.B, U2.P0.20
- net DTR: now also C9.1, U2.!DTR; no longer C14.1, U5.!DTR
- net FRST: now also U1.P0.22; no longer U2.P0.22
- net FT3V3: now also U2.3V3OUT; no longer U5.3V3OUT
- net GND: now also C1.2, C10.1, C13.1, C15.1, C2.1, C3.1, C4.2, C6.1, C8.2, CHRG1.VSS, DEBUG1.GND@3, DEBUG1.GND@5, DEBUG1.GNDDTCT, DEBUG1.KEY, J1.1, J2.3, LDO1.GND, LED1.C, LED2.C, R12.1, R14.2, R5.1, R8.1, SD1.GND, SD1.GND1, SD1.VSS, SW2.A, SW3.3, SW3.4, U1.GND@1, U1.GND@2, U1.GND@3, U1.GND@4, U2.GND@16, U2.GND@6, USB1.GND; no longer C10.2, C16.1, C19.1, C2.2, C20.2, C21.1, C22.1, C23.2, C24.1, C6.2, C8.1, C9.2, CHRG2.VSS, CORTEX1.GND@3, CORTEX1.GND@5, CORTEX1.GNDDTCT, CORTEX1.KEY, J2.1, LDO2.GND, LED3.C, LED4.C, R11.1, R14.1, R15.1, R6.1, R7.2, SD2.GND, SD2.GND1, SD2.VSS, SW2.3, SW2.4, SW3.A, SW5.3, SW5.4, U2.GND@1, U2.GND@2, U2.GND@3, U2.GND@4, U4.VSS, U5.GND@16, U5.GND@6, USB2.GND
- net LED1: now also R4.2, U1.P0.17; no longer R3.2, U2.P0.17
- net LED2: now also R6.2, U1.P0.19; no longer R4.2, U2.P0.19
- net MISO: now also SD1.DATA_OUT, U1.P0.14; no longer SD2.DATA_OUT, U2.P0.14
- net MOSI: now also SD1.DATA_IN, U1.P0.13; no longer SD2.DATA_IN, U2.P0.13
- net N$1: now also R12.2; no longer R6.2
- net N$10: now also LED2.A, R6.1; no longer LED4.A, R4.1
- net N$11: now also U1.DCC; no longer U2.DCC
- net N$12: now also C1.1, U1.DEC4; no longer C7.1, U2.DEC4
- net N$13: now also C13.2; no longer C16.2
- net N$14: now also DEBUG1.NC/TDI; no longer CORTEX1.NC/TDI
- net N$15: now also C15.2; no longer C18.2
- net N$16: now also C4.1, U1.P0.01/XL2; no longer C9.1, U2.P0.01/XL2
- net N$17: now also CHRG1.PROG, R5.2; no longer CHRG2.PROG, R11.2
- net N$2: now also R14.1; no longer R7.1
- net N$23: now also R10.2, U2.USBDM; no longer R17.2, U5.USBDM
- net N$24: now also R11.2, U2.USBDP; no longer R18.2, U5.USBDP
- net N$25: now also LED3.C, R13.2; no longer LED5.C, R19.2
- net N$26: now also LED4.C, R15.2; no longer LED6.C, R20.2
- net N$3: now also C16.2; no longer C13.2
- net N$4: now also C3.2, U1.P0.00/XL1; no longer C8.2, U2.P0.00/XL1
- net N$5: now also C16.1; no longer C13.1
- net N$7: now also C14.2; no longer C15.2
- net N$8: now also C14.1; no longer C15.1
- net N$9: now also LED1.A, R4.1; no longer LED3.A, R3.1
- net P0.09/NFC1: now also U1.P0.09; no longer C11.1, U2.P0.09
- net P0.10/NFC2: now also U1.P0.10; no longer C10.1, U2.P0.10
- net RESET: now also C9.2, D3.A, DEBUG1.!RESET, R9.1, U1.P0.21/RESET; no longer C14.2, CORTEX1.!RESET, D1.A, R5.1, U2.P0.21/RESET
- net RXD.FT: now also R17.1, U2.RXD; no longer R2.1, U5.RXD
- net RXD.NRF: now also R16.2, U1.P0.08; no longer R1.2, U2.P0.08
- net RXLED: now also R13.1, U2.CBUS1; no longer R19.1, U5.CBUS1
- net SCK: now also SD1.SCLK, U1.P0.12; no longer SD2.SCLK, U2.P0.12
- net SCL: now also J2.2, R2.1, U1.P0.26; no longer R9.1, U2.P0.26, U4.SCL
- net SDA: now also J2.1, R1.1, U1.P0.25; no longer R8.1, U2.P0.25, U4.SDA
- net SWCLK: now also DEBUG1.SWDCLK/TCK, U1.SWDCLK; no longer CORTEX1.SWDCLK/TCK, U2.SWDCLK
- net SWDIO: now also DEBUG1.SWDIO/TMS, U1.SWDIO; no longer CORTEX1.SWDIO/TMS, U2.SWDIO
- net SWO: now also DEBUG1.SWO/TDO, U1.P0.18/SWO; no longer CORTEX1.SWO/TDO, U2.P0.18/SWO
- net TXD.FT: now also R16.1, U2.TXD; no longer U5.TXD
- net TXD.NRF: now also R17.2, U1.P0.06; no longer R2.2, U2.P0.06
- net TXLED: now also R15.1, U2.CBUS2; no longer R20.1, U5.CBUS2
- net USB+: now also C11.1, R11.1, USB1.D+; no longer C23.1, R18.1, USB2.D+
- net USB-: now also C10.2, R10.1, USB1.D-; no longer C24.2, R17.1, USB2.D-
- net VIN: now also C6.2, CHRG1.VIN, D1.C, D2.C, LDO1.EN, LDO1.IN, R3.2; no longer C21.2, CHRG2.VIN, D4.C, D5.C, LDO2.EN, LDO2.IN, R12.2
- net VLIPO: now also C8.1, CHRG1.VBAT, D1.A, J1.2, R7.2; no longer C20.1, CHRG2.VBAT, D4.A, J2.2, R13.2
- net V_USB: now also D2.A, U2.VCC, USB1.V+; no longer D5.A, U5.VCC, USB2.V+
Other:
- note added: "0 ohm resistors in case RX and TX are mixed up"
- note added: "Connection to lower board"
- note added: "Diode switch from LiPo Power to USB when USB is connected The USB power can charge the battery"
- note added: "Headers connecting top to bottom boards"
- note added: "Power Management D27/CHRG.STATUS Iinput) A7/BATT (Input) PPG Circuit D29/LED.CTRL (Output) A4/PPG (Input) OLED Pins D3/RESET.OLED (Output) D4/DC.OLED (Output) D16/CS.OLED (Output) SD Card Pins D5/CD1 (Input) D7/SD.CS (Output) Button Pins D11/SW1 (Input) D15/SW2 (Input)"
- note added: "R5 sets charge current I_charge = 1000V/R4 per MCP3831datasheet"
- note added: "Voltage divider useed to monitor battery voltage"
- note removed: "Back-up battery if desired"
- note removed: "I2C Address = 0x68h"
- note removed: "Power Management D27/CHRG.STATUS Iinput) A4/BATT (Input) PPG Circuit D29/LED.CTRL (Output) A7/PPG (Input) OLED Pins D3/RESET.OLED (Output) D4/DC.OLED (Output) D16/CS.OLED (Output) SD Card Pins D5/CD1 (Input) D7/SD.CS (Output) Button Pins D11/SW1 (Input) D15/SW2 (Input)"
- note removed: "Real-Time Clock"
- moved on the sheet: C10, C11, C12, C13, C14, C15, C16, C17, C18, C2, C5, C6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

Commit message: Small changes
Parts:
- renumbered SW4 to RESET
Changed lines of the file:
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@@
 <part name="SW2" library="LinnesLab-Switches" deviceset="SPST-PTS830GG140-COPY" device=".1-3" package3d_urn="urn:adsk.eagle:package:18580190/2"/>
 <part name="GND30" library="LinnesLab-Symbols" deviceset="GND" device=""/>
-<part name="SW4" library="LinnesLab-Switches" deviceset="SPST-PTS830GG140-COPY" device=".1-3" package3d_urn="urn:adsk.eagle:package:18580190/2"/>
+<part name="RESET" library="LinnesLab-Switches" deviceset="SPST-PTS830GG140-COPY" device=".1-3" package3d_urn="urn:adsk.eagle:package:18580190/2"/>
 <part name="U1" library="LinnesLab-Microcontrollers" deviceset="NRF52832_MODULE_MDBT42" device="" override_package3d_urn="urn:adsk.eagle:package:18593121/2" override_package_urn="urn:adsk.eagle:footprint:18593122/1"/>
 <part name="LED1" library="LinnesLab-LED" deviceset="LED" device="0603" package3d_urn="urn:adsk.eagle:package:18593052/2" value="RED"/>
@@
 <attribute name="VALUE" x="185.42" y="251.206" size="1.778" layer="96" align="top-center"/>
 </instance>
-<instance part="SW4" gate="G$1" x="373.38" y="127" smashed="yes">
+<instance part="RESET" gate="G$1" x="373.38" y="127" smashed="yes">
 <attribute name="NAME" x="370.84" y="124.46" size="1.27" layer="95"/>
 <attribute name="VALUE" x="370.84" y="121.92" size="1.27" layer="96"/>
@@
 <wire x1="381" y1="127" x2="381" y2="124.46" width="0.1524" layer="91"/>
 <pinref part="GND28" gate="G$1" pin="GND"/>
-<pinref part="SW4" gate="G$1" pin="B"/>
+<pinref part="RESET" gate="G$1" pin="B"/>
 </segment>
 <segment>
@@
 <wire x1="365.76" y1="127" x2="368.3" y2="127" width="0.1524" layer="91"/>
 <label x="365.76" y="127" size="1.27" layer="95" rot="R180" xref="yes"/>
-<pinref part="SW4" gate="G$1" pin="A"/>
-</segment>
-<segment>
+<pinref part="RESET" gate="G$1" pin="A"/>
+</segment>
+<segment>
